File: Vehicle/Schematics/robo-chopper.sch (KiCad schematic (older format))
At the start: 76 parts

Commit message: Removes encoders. Removes accelerometer. Removes gyro. Adds 2 Ping inputs. Adds 4 Servo outputs. Adds 9DOF INU input. Adds another LED status.
TODO:
Resize servo headers.
Design power supply circuitry.
Move compass to propeller according to spec.
Isolate servo and speed controller PWMs.
Adds 4 banks of tricolor LEDs.
Parts:
- removed P? (x4): CONN_2X2, symbol CONN_2X2
- removed P?: CONN_7, symbol CONN_7
- removed P?: CONN_6, symbol CONN_6
- added D?: LED, symbol LED
- added K? (x9): CONN_3, symbol CONN_3
- added P? (x2): CONN_7, symbol CONN_7
- added R?: 270, symbol RES
Connections:
- net labels added: INU_RX, INU_TX, MOTOR_PWM5, MOTOR_PWM6, MOTOR_PWM7, MOTOR_PWM8, PING5_ANA, PING5_PWM, PING5_RX, PING6_ANA, PING6_PWM, PING6_RX, PROP_SPI_CLK, PROP_SPI_CSP, PROP_SPI_DIO, RX_INU, SERVO_PWM1, SERVO_PWM2, SERVO_PWM3, SERVO_PWM4, SEVRO_PWM3, STAT_LED4, TX_INU
- net labels removed: ACC_XOUT, ACC_YOUT, ACC_ZOUT, ENCODER1A, ENCODER1B, ENCODER2A, ENCODER2B, ENCODER3A, ENCODER3B, ENCODER4A, ENCODER4B, GYRO_XOUT, GYRO_YOUT
- wire segments 384 -> 414
Other:
- note added: "9DOF RAZOR INU"
- note added: "SERVO OUTPUTS"
- note added: "YELLOW"
- note removed: "ACCELEROMETER"
- note removed: "ENCODER INPUTS"
- note removed: "GYROSCOPE"
- moved on the sheet: C?, CN?, EC?, JK?, L?, R?, SOK?, T?, U?

Commit message: Adds 5V, 6V, and 3.3V power supply circuitry.
Parts:
- removed U?: BOOST_CONVERTER, symbol BOOST_CONVERTER
- added C? (x2): .01 uF, symbol CAP
- added C? (x2): .1 uF, symbol CAP
- added C? (x2): 330 uF, symbol CAP_E
- added C? (x4): 4.7 uF, symbol CAP
- added C? (x2): 10 uF, symbol CAP_E
- added C? (x5): 0.1 uF, symbol CAP
- added D? (x2): MBRA340T3G, symbol DIODESCH
- added L? (x2): 22 uH, symbol IND
- added R?: 30.9 K, symbol RES
- added R? (x2): 10 K, symbol RES
- added R?: 39.2 K, symbol RES
- added U? (x2): TPS5431DDA, symbol TPS5431DDA
Connections:
- net labels added: +6V, +BATT, AGND
- wire segments 414 -> 481
Other:
- moved on the sheet: U?

Commit message: Adds work completed last weekend at D's apartment.
Parts:
- removed P? (x7): CONN_7, symbol CONN_7
- added C? (x4): 0.1 uF, symbol CAP
- added D?: LED, symbol LED
- added K? (x15): CONN_3, symbol CONN_3
- added R?: 270, symbol RES
- added R? (x2): 10 K, symbol RES
- added SW?: SWITCH, symbol SWITCH
- added U? (x2): TXB0108PWR, symbol TXB0108PWR
Connections:
- net labels added: PWM5_LD1, PWM6_LD2, PWM7_LD3, PWM8_LD4, SOM_AN0, SOM_AN1, SOM_AN2, SOM_AN3
- net labels removed: PING0_PWM, PING0_RX, PING1_PWM, PING1_RX, PING2_PWM, PING2_RX, PING3_PWM, PING3_RX, PING4_PWM, PING4_RX, PING5_PWM, PING5_RX, PING6_PWM, PING6_RX, STAT_LED1, STAT_LED2, STAT_LED3, STAT_LED4
- wire segments 481 -> 581
Other:
- note added: "ANALOG EXPANSION"
- moved on the sheet: C?, R?, U?

Commit message: Adds power input terminals with overcurrent and reverse voltage protection. Adds 4 BlinkM module connectors. Adds reference designators.
Schematic is ready for internal design review and PCB artwork.
Parts:
- added D1: ZENER, symbol ZENER
- added F1: FUSE, symbol FUSE
- added P1: CONN_2, symbol CONN_2
- added P4, P5, P6, P7: CONN_4, symbol CONN_4
- added R22, R23, R24, R25: 4.7 K, symbol RES
- gave numbers to parts that had none: 128
Connections:
- net labels added: I2C_SCL_PROP, I2C_SDA_PROP
- net labels removed: AGND
- wire segments 581 -> 621
Other:
- note added: "BATTERY TERMINAL"
- note added: "BLINKM LED MODULES"
